File: hardware/HEVEN_Cluster_RevB/HEVEN_Cluster_RevB.kicad_pcb (KiCad board)
At the start: 2 copper layers, 350 x 90 mm, 49 parts

Commit message: fix(hardware): reroute Cluster RevB R2
Parts:
- moved R_LCD_MOSI 12.8 mm to (225.0, 12.0)
- moved R_LCD_MISO 12.2 mm to (225.0, 15.0)
- moved R_LCD_SCK 11.7 mm to (225.0, 18.0)
- moved R_LCD_CS 11.2 mm to (225.0, 21.0)
- moved R_LCD_DC 10.8 mm to (225.0, 24.0)
- moved R_LCD_RST 10.4 mm to (225.0, 27.0)
- moved R_TOUCH_CS 10.2 mm to (225.0, 30.0)
- moved U_ESP 3.00 mm to (260.0, 45.0)
- moved C_CAN 2.50 mm to (280.0, 40.5)
- turned C_PWR_HF to 180 degrees
- turned D_TVS5 to 180 degrees
Routing:
- net 5V_SYS: track 278.9 -> 193.8 mm, vias 0 -> 1
- net TOUCH_CS: track 187.6 -> 109.1 mm, vias 0 -> 3
- net LCD_MOSI_MCU: track 127.3 -> 58.1 mm, vias 2 -> 1
- net LCD_RST: track 209.6 -> 143.1 mm
- net LCD_MOSI: track 195.9 -> 136.7 mm, vias 0 -> 1
- net WARNING_DETAIL: track 75.5 -> 22.1 mm, vias 2 -> 0
- net LCD_MISO: track 182.3 -> 133.2 mm, vias 0 -> 3
- net TOUCH_CS_MCU: track 114.8 -> 72.6 mm, vias 2 -> 0
- net PADDOCK: track 298.2 -> 256.2 mm, vias 2 -> 0
- net LCD_CS: track 166.9 -> 125.6 mm
- net LCD_DC: track 174.1 -> 137.6 mm
- net LCD_SCK: track 175.7 -> 149.1 mm, vias 2 -> 1
- net LCD_SCK_MCU: track 107.2 -> 130.1 mm, vias 2 -> 9
- net 3V3: track 115.1 -> 137.5 mm, vias 0 -> 1
- net LCD_MISO_MCU: track 22.8 -> 42.6 mm, vias 0 -> 2
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Other:
- board text removed: "ESP32 USB-C ACCESS / ANTENNA NOTCH"

Commit message: fix(hardware): reroute Cluster RevB R3
Parts:
- moved H6 3.00 mm to (238.0, 85.0)
Connections:
- U_ESP pad 14: GND -> (no net)
Routing:
- net 5V_SYS: track 193.8 -> 193.7 mm, vias 1 -> 0
Other:
- board text added: "HEVEN CLUSTER REV.B R3 | 350 x 90 mm | 2026-08-01"
- board text removed: "HEVEN CLUSTER REV.B | 350 x 90 mm | 2026-08-01"
Changed lines of the file:
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@@
 	(footprint "HEVEN_Cluster_RevB:MountingHole_M3"
 		(layer "F.Cu")
-		(at 235 85)
+		(at 238 85)
 		(property "Reference" "H6"
 			(at 0 -4 0)
@@
 			(layers "*.Cu" "*.Mask")
 			(remove_unused_layers no)
-			(net "GND")
 		)
 		(pad "15" thru_hole circle
@@
 	)
 	(gr_text "RIGHT PANEL RESERVED - TEMPORARY HOLES ONLY"
-		(at 320 84 0)
+		(at 320 80 0)
 		(layer "F.SilkS")
 		(effects
@@
 		)
 	)
-	(gr_text "HEVEN CLUSTER REV.B  |  350 x 90 mm  |  2026-08-01"
+	(gr_text "HEVEN CLUSTER REV.B R3  |  350 x 90 mm  |  2026-08-01"
 		(at 175 87 0)
 		(layer "F.SilkS")
@@
 		(net "5V_SYS")
 	)
-	(via
-		(at 248.5 68)
-		(size 0.9)
-		(drill 0.4)
-		(layers "F.Cu" "B.Cu")
-		(net "5V_SYS")
-	)
 	(segment
 		(start 267 68)
-		(end 248.5 68)
+		(end 248.57 67.86)
 		(width 0.6)
 		(layer "B.Cu")
@@
 			(thermal_gap 0.35)
 			(thermal_bridge_width 0.4)
-			(island_removal_mode 1)
+			(island_removal_mode 0)
 		)
 		(polygon
@@
 			(thermal_gap 0.35)
 			(thermal_bridge_width 0.4)
-			(island_removal_mode 1)
+			(island_removal_mode 0)
 		)
 		(polygon

Commit message: fix(hardware): connect RevB ground zones R4
Routing:
- net GND: track 0.00 -> 6.75 mm, vias 0 -> 25

Commit message: fix(hardware): resolve RevB footprint library warnings R5
Parts:
- C_PWR_HF, D_TVS5: footprint HEVEN_Cluster_RevB:C_0805 -> HEVEN_Cluster_RevB:C_0805_R180
- turned C_PWR_HF to 0 degrees
- turned D_TVS5 to 0 degrees
Routing:
- net GND: track 6.75 -> 32.1 mm, vias 25 -> 31
Changed lines of the file:
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@@
 		(embedded_fonts no)
 	)
-	(footprint "HEVEN_Cluster_RevB:C_0805"
+	(footprint "HEVEN_Cluster_RevB:C_0805_R180"
 		(layer "B.Cu")
-		(at 266 82 180)
+		(at 266 82)
 		(duplicate_pad_numbers_are_jumpers yes)
 		(property "Reference" "C_PWR_HF"
@@
 		)
 		(pad "1" smd roundrect
+			(at 1.1 0 0)
+			(size 1.2 1.4)
+			(layers "B.Cu" "B.Paste" "B.Mask")
+			(roundrect_rratio 0.2)
+			(net "5V_SYS")
+)
+		(pad "2" smd roundrect
 			(at -1.1 0 0)
-			(size 1.2 1.4)
-			(layers "B.Cu" "B.Paste" "B.Mask")
-			(roundrect_rratio 0.2)
-			(net "5V_SYS")
-)
-		(pad "2" smd roundrect
-			(at 1.1 0 0)
 			(size 1.2 1.4)
 			(layers "B.Cu" "B.Paste" "B.Mask")
@@
 		(embedded_fonts no)
 	)
-	(footprint "HEVEN_Cluster_RevB:C_0805"
+	(footprint "HEVEN_Cluster_RevB:C_0805_R180"
 		(layer "B.Cu")
-		(at 266 78 180)
+		(at 266 78)
 		(duplicate_pad_numbers_are_jumpers yes)
 		(property "Reference" "D_TVS5"
@@
 		)
 		(pad "1" smd roundrect
+			(at 1.1 0 0)
+			(size 1.2 1.4)
+			(layers "B.Cu" "B.Paste" "B.Mask")
+			(roundrect_rratio 0.2)
+			(net "5V_SYS")
+)
+		(pad "2" smd roundrect
 			(at -1.1 0 0)
-			(size 1.2 1.4)
-			(layers "B.Cu" "B.Paste" "B.Mask")
-			(roundrect_rratio 0.2)
-			(net "5V_SYS")
-)
-		(pad "2" smd roundrect
-			(at 1.1 0 0)
 			(size 1.2 1.4)
 			(layers "B.Cu" "B.Paste" "B.Mask")
@@
 	(via (at 335 75) (size 0.9) (drill 0.4)
 		(layers "F.Cu" "B.Cu") (net "GND"))
+	(segment (start 256.100000 78.000000) (end 255.350000 76.700962)
+		(width 0.5) (layer "B.Cu") (net "GND"))
+	(segment (start 256.100000 82.000000) (end 257.600000 82.000000)
+		(width 0.5) (layer "B.Cu") (net "GND"))
+	(segment (start 271.100000 82.000000) (end 272.600000 82.000000)
+		(width 0.5) (layer "B.Cu") (net "GND"))
+	(segment (start 264.900000 82.000000) (end 265.000000 80.000000)
+		(width 0.5) (layer "B.Cu") (net "GND"))
+	(segment (start 264.900000 78.000000) (end 265.000000 80.000000)
+		(width 0.5) (layer "B.Cu") (net "GND"))
+	(segment (start 278.000000 30.950000) (end 279.448889 30.561771)
+		(width 0.5) (layer "B.Cu") (net "GND"))
+	(segment (start 281.100000 40.500000) (end 281.850000 41.799038)
+		(width 0.5) (layer "B.Cu") (net "GND"))
+	(segment (start 291.100000 40.000000) (end 292.600000 40.000000)
+		(width 0.5) (layer "B.Cu") (net "GND"))
+	(segment (start 282.300000 34.365000) (end 283.400000 34.800000)
+		(width 0.3) (layer "B.Cu") (net "GND"))
+	(segment (start 283.400000 34.800000) (end 286.800000 37.800000)
+		(width 0.3) (layer "B.Cu") (net "GND"))
+	(segment (start 286.800000 37.800000) (end 290.600000 38.000000)
+		(width 0.3) (layer "B.Cu") (net "GND"))
+	(segment (start 290.600000 38.000000) (end 292.600000 40.000000)
+		(width 0.3) (layer "B.Cu") (net "GND"))
+	(via (at 255.350000 76.700962) (size 0.9) (drill 0.4)
+		(layers "F.Cu" "B.Cu") (net "GND"))
+	(via (at 257.600000 82.000000) (size 0.9) (drill 0.4)
+		(layers "F.Cu" "B.Cu") (net "GND"))
+	(via (at 272.600000 82.000000) (size 0.9) (drill 0.4)
+		(layers "F.Cu" "B.Cu") (net "GND"))
+	(via (at 279.448889 30.561771) (size 0.9) (drill 0.4)
+		(layers "F.Cu" "B.Cu") (net "GND"))
+	(via (at 281.850000 41.799038) (size 0.9) (drill 0.4)
+		(layers "F.Cu" "B.Cu") (net "GND"))
+	(via (at 292.600000 40.000000) (size 0.9) (drill 0.4)
+		(layers "F.Cu" "B.Cu") (net "GND"))
 	(zone (net "GND") (layer "F.Cu") (hatch edge 0.5)
